File: docs/pi_flux_r3_wiring.kicad_sch (KiCad schematic)
At the start: 17 parts, among them J1 4x 21700 pack (4S), J10 Wired USB keyboard, J11 Panasonic ML-2020, J12 FireBeetle 2 ESP32-UE, J13 1.3 inch OLED 0x3C, J14 BME688 0x76/0x77, J15 DS3231 RTC 0x68, J16 Trackball 0x0A (optional), J17 PBS-33B status button, J2 Foldable solar panel, J3 Hand crank generator, J4 Sealed USB-C port, J5 MPPT / charger, J6 Waveshare UPS HAT (E), J7 Raspberry Pi 5, J8 DFR0550-V2 5 inch DSI, J9 Seeed M.2 BASE + 1TB

Commit message: Retarget wiring diagrams and schematic for the r3 build
Rename the KiCad schematic, PDF, PNG, SVG and netlist CSV to pi_flux_r3_*;
rev 2 carries the r3 title and a Phistone 2.4G dongle block (J10) on the
USB_KEYBOARD net. The r2-only trackball J16 is marked DNP (crossed out) and
the notes state that r3 uses no trackball.

Regenerate the Graphviz data/power diagrams: the keyboard node is now the
Phistone (dongle or Bluetooth, no cable, own battery), the trackball node is
gone, and the power diagram carries an r3 keyboard-power note. WIRING.md
documents the wireless keyboard link, drops the keyboard from the common-
ground rule, and adds an r3 keyboard-link check; README points at the r3
artifacts. ERC is clean apart from lib_symbol_issues.
Parts:
- J10: value Wired USB keyboard -> Phistone 2.4G dongle
- J16: value Trackball 0x0A (optional) -> Trackball 0x0A (r2 only); now not fitted; now left out of the parts list
Other:
- note added: "R3 keyboard: the case holds only the Phistone 2.4G dongle (J10) in a Pi USB-A port. Bluetooth option: no dongle, no wire."
- note added: "USB_FB_SERIAL: FireBeetle USB-C to Pi USB-A, data-only preferred. Trackball is r2-only; r3 uses none."
- note removed: "USB_FB_SERIAL: FireBeetle USB-C to Pi USB-A, data-only preferred. Trackball firmware pending."
- title: Pi Fluks r2 - wiring / connections -> Pi Fluks r3 - wiring / connections
Changed lines of the file:
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@@
   (paper "A3")
   (title_block
-    (title "Pi Fluks r2 - wiring / connections")
-    (date "2026-10-19")
-    (rev "1")
+    (title "Pi Fluks r3 - wiring / connections")
+    (date "2026-10-20")
+    (rev "2")
     (company "Pi Fluks")
   )
@@
     (pin "2")
     (instances
-      (project "pi_flux_r2_wiring"
+      (project "pi_flux_r3_wiring"
         (path "/9545ffa8-4da6-4e23-961a-0f1b69dedae2"
           (reference "J1")
@@
     (pin "2")
     (instances
-      (project "pi_flux_r2_wiring"
+      (project "pi_flux_r3_wiring"
         (path "/9545ffa8-4da6-4e23-961a-0f1b69dedae2"
           (reference "J2")
@@
     (pin "2")
     (instances
-      (project "pi_flux_r2_wiring"
+      (project "pi_flux_r3_wiring"
         (path "/9545ffa8-4da6-4e23-961a-0f1b69dedae2"
           (reference "J3")
@@
     (pin "2")
     (instances
-      (project "pi_flux_r2_wiring"
+      (project "pi_flux_r3_wiring"
         (path "/9545ffa8-4da6-4e23-961a-0f1b69dedae2"
           (reference "J4")
@@
     (pin "4")
     (instances
-      (project "pi_flux_r2_wiring"
+      (project "pi_flux_r3_wiring"
         (path "/9545ffa8-4da6-4e23-961a-0f1b69dedae2"
           (reference "J5")
@@
     (pin "8")
     (instances
-      (project "pi_flux_r2_wiring"
+      (project "pi_flux_r3_wiring"
         (path "/9545ffa8-4da6-4e23-961a-0f1b69dedae2"
           (reference "J6")
@@
     (pin "8")
     (instances
-      (project "pi_flux_r2_wiring"
+      (project "pi_flux_r3_wiring"
         (path "/9545ffa8-4da6-4e23-961a-0f1b69dedae2"
           (reference "J7")
@@
     (pin "2")
     (instances
-      (project "pi_flux_r2_wiring"
+      (project "pi_flux_r3_wiring"
         (path "/9545ffa8-4da6-4e23-961a-0f1b69dedae2"
           (reference "J8")
@@
     (pin "2")
     (instances
-      (project "pi_flux_r2_wiring"
+      (project "pi_flux_r3_wiring"
         (path "/9545ffa8-4da6-4e23-961a-0f1b69dedae2"
           (reference "J9")
@@
       (effects (font (size 1.8 1.8)) (justify left))
     )
-    (property "Value" "Wired USB keyboard"
+    (property "Value" "Phistone 2.4G dongle"
       (at 201.18 153.13 0)
       (show_name no)
@@
     (pin "2")
     (instances
-      (project "pi_flux_r2_wiring"
+      (project "pi_flux_r3_wiring"
         (path "/9545ffa8-4da6-4e23-961a-0f1b69dedae2"
           (reference "J10")
@@
     (pin "2")
     (instances
-      (project "pi_flux_r2_wiring"
+      (project "pi_flux_r3_wiring"
         (path "/9545ffa8-4da6-4e23-961a-0f1b69dedae2"
           (reference "J11")
@@
     (pin "8")
     (instances
-      (project "pi_flux_r2_wiring"
+      (project "pi_flux_r3_wiring"
         (path "/9545ffa8-4da6-4e23-961a-0f1b69dedae2"
           (reference "J12")
@@
     (pin "4")
     (instances
-      (project "pi_flux_r2_wiring"
+      (project "pi_flux_r3_wiring"
         (path "/9545ffa8-4da6-4e23-961a-0f1b69dedae2"
           (reference "J13")
@@
     (pin "4")
     (instances
-      (project "pi_flux_r2_wiring"
+      (project "pi_flux_r3_wiring"
         (path "/9545ffa8-4da6-4e23-961a-0f1b69dedae2"
           (reference "J14")
@@
     (pin "4")
     (instances
-      (project "pi_flux_r2_wiring"
+      (project "pi_flux_r3_wiring"
         (path "/9545ffa8-4da6-4e23-961a-0f1b69dedae2"
           (reference "J15")
@@
     (body_style 1)
     (exclude_from_sim no)
-    (in_bom yes)
-    (on_board yes)
-    (in_pos_files yes)
-    (dnp no)
+    (in_bom no)
+    (on_board yes)
+    (in_pos_files yes)
+    (dnp yes)
     (property "Reference" "J16"
       (at 331.99 194.85 0)
@@
       (effects (font (size 1.8 1.8)) (justify left))
     )
-    (property "Value" "Trackball 0x0A (optional)"
+    (property "Value" "Trackball 0x0A (r2 only)"
       (at 331.99 198.85 0)
       (show_name no)
@@
     (pin "4")
     (instances
-      (project "pi_flux_r2_wiring"
+      (project "pi_flux_r3_wiring"
         (path "/9545ffa8-4da6-4e23-961a-0f1b69dedae2"
           (reference "J16")
@@
     (pin "2")
     (instances
-      (project "pi_flux_r2_wiring"
+      (project "pi_flux_r3_wiring"
         (path "/9545ffa8-4da6-4e23-961a-0f1b69dedae2"
           (reference "J17")
@@
   (text "CHG_VBUS: solar and crank share the one sealed port. BATT_4S: 4x21700 series, fuse positive."
     (at 20 262 0) (effects (font (size 2 2)) (justify left)))
-  (text "USB_FB_SERIAL: FireBeetle USB-C to Pi USB-A, data-only preferred. Trackball firmware pending."
+  (text "USB_FB_SERIAL: FireBeetle USB-C to Pi USB-A, data-only preferred. Trackball is r2-only; r3 uses none."
     (at 20 268 0) (effects (font (size 2 2)) (justify left)))
+  (text "R3 keyboard: the case holds only the Phistone 2.4G dongle (J10) in a Pi USB-A port. Bluetooth option: no dongle, no wire."
+    (at 20 274 0) (effects (font (size 2 2)) (justify left)))
   (sheet_instances
     (path "/" (page "1"))
