File: docs/ktemata_r3_wiring.kicad_sch (KiCad schematic)
At the start: 17 parts, among them J1 4x 21700 pack (4S), J10 Phistone 2.4G dongle, J11 Panasonic ML-2020, J12 FireBeetle 2 ESP32-UE, J13 1.3 inch OLED 0x3C, J14 BME688 0x76/0x77, J15 DS3231 RTC 0x68, J16 Trackball 0x0A (r2 only), J17 PBS-33B status button, J2 Foldable solar panel, J3 Hand crank generator, J4 Sealed USB-C port, J5 MPPT / charger, J6 Waveshare UPS HAT (E), J7 Raspberry Pi 5, J8 DFR0550-V2 5 inch DSI, J9 Seeed M.2 BASE + 1TB

Commit message: Rename the project to Ktemata
Ktemata (Greek kappa-tau-eta-mu-alpha-tau-alpha, "possessions") comes from Thucydides'
kappa-tau-eta-mu-alpha epsilon-sigma alpha-epsilon-iota, "a possession for all time".
The device is an offline library that survives the loss of power and networking,
which is what that phrase claims for a written record.

- Wordmark: the face and the bottom shell now emboss Kappa-Tau-Eta-Mu-Alpha-Tau-Alpha
  instead of the old pi-FLUKS/AI mark; the motto becomes the Thucydides phrase
  (Liberation Sans has the Greek glyphs, so no new font dependency).
- Files: stl/ and renders/ are ktemata_*; the KiCad schematic, PDF, PNG, SVG and CSV
  are ktemata_r3_* (regenerated with kicad-cli, so the title block reads Ktemata and
  the embedded symbols are Ktemata:*).
- Tools: export.py writes ktemata_* names; render.py views follow.
- Docs: README opens with a paragraph on the name; AGENTS/BOM/R3/R4/WIRING/
  POCKETTERM35/firmware docs and the firmware banner/JSON message updated.

Geometry is unchanged: parts export with bad edges: 0 and the interference checks pass.
The only remaining "Pi_Flux" string is the filename of the original build-guide PDF,
which is an external asset referenced as-is.
Parts:
- J1: symbol PiFlux:BATT -> Ktemata:BATT
- J10: symbol PiFlux:KEYBOARD -> Ktemata:KEYBOARD
- J11: symbol PiFlux:PI_RTC -> Ktemata:PI_RTC
- J12: symbol PiFlux:FB -> Ktemata:FB
- J13: symbol PiFlux:OLED -> Ktemata:OLED
- J14: symbol PiFlux:BME -> Ktemata:BME
- J15: symbol PiFlux:DS3231 -> Ktemata:DS3231
- J16: symbol PiFlux:TRACK -> Ktemata:TRACK
- J17: symbol PiFlux:BUTTON -> Ktemata:BUTTON
- J2: symbol PiFlux:SOLAR -> Ktemata:SOLAR
- J3: symbol PiFlux:CRANK -> Ktemata:CRANK
- J4: symbol PiFlux:CHG_PORT -> Ktemata:CHG_PORT
- J5: symbol PiFlux:MPPT -> Ktemata:MPPT
- J6: symbol PiFlux:UPS -> Ktemata:UPS
- J7: symbol PiFlux:PI5 -> Ktemata:PI5
- J8: symbol PiFlux:DISPLAY -> Ktemata:DISPLAY
- J9: symbol PiFlux:NVME -> Ktemata:NVME
Other:
- company: Pi Fluks -> Ktemata
- title: Pi Fluks r3 - wiring / connections -> Ktemata r3 - wiring / connections
Changed lines of the file:
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@@
   (paper "A3")
   (title_block
-    (title "Pi Fluks r3 - wiring / connections")
+    (title "Ktemata r3 - wiring / connections")
     (date "2026-10-20")
     (rev "2")
-    (company "Pi Fluks")
-  )
-  (symbol
-    (lib_id "PiFlux:BATT")
+    (company "Ktemata")
+  )
+  (symbol
+    (lib_id "Ktemata:BATT")
     (at 59.69 55.88 0)
     (unit 1)
@@
     (pin "2")
     (instances
-      (project "pi_flux_r3_wiring"
+      (project "ktemata_r3_wiring"
         (path "/9545ffa8-4da6-4e23-961a-0f1b69dedae2"
           (reference "J1")
@@
   (label "BATT_4S_N" (at 44.45 58.42 180) (effects (font (size 2 2)) (justify right bottom)))
   (symbol
-    (lib_id "PiFlux:SOLAR")
+    (lib_id "Ktemata:SOLAR")
     (at 59.69 85.09 0)
     (unit 1)
@@
     (pin "2")
     (instances
-      (project "pi_flux_r3_wiring"
+      (project "ktemata_r3_wiring"
         (path "/9545ffa8-4da6-4e23-961a-0f1b69dedae2"
           (reference "J2")
@@
   (label "GND" (at 44.45 87.63000000000001 180) (effects (font (size 2 2)) (justify right bottom)))
   (symbol
-    (lib_id "PiFlux:CRANK")
+    (lib_id "Ktemata:CRANK")
     (at 59.69 110.49 0)
     (unit 1)
@@
     (pin "2")
     (instances
-      (project "pi_flux_r3_wiring"
+      (project "ktemata_r3_wiring"
         (path "/9545ffa8-4da6-4e23-961a-0f1b69dedae2"
           (reference "J3")
@@
   (label "GND" (at 44.45 113.03 180) (effects (font (size 2 2)) (justify right bottom)))
   (symbol
-    (lib_id "PiFlux:CHG_PORT")
+    (lib_id "Ktemata:CHG_PORT")
     (at 59.69 135.89 0)
     (unit 1)
@@
     (pin "2")
     (instances
-      (project "pi_flux_r3_wiring"
+      (project "ktemata_r3_wiring"
         (path "/9545ffa8-4da6-4e23-961a-0f1b69dedae2"
           (reference "J4")
@@
   (label "GND" (at 44.45 138.42999999999998 180) (effects (font (size 2 2)) (justify right bottom)))
   (symbol
-    (lib_id "PiFlux:MPPT")
+    (lib_id "Ktemata:MPPT")
     (at 59.69 170.18 0)
     (unit 1)
@@
     (pin "4")
     (instances
-      (project "pi_flux_r3_wiring"
+      (project "ktemata_r3_wiring"
         (path "/9545ffa8-4da6-4e23-961a-0f1b69dedae2"
           (reference "J5")
@@
   (label "GND" (at 44.45 175.26000000000002 180) (effects (font (size 2 2)) (justify right bottom)))
   (symbol
-    (lib_id "PiFlux:UPS")
+    (lib_id "Ktemata:UPS")
     (at 59.69 215.9 0)
     (unit 1)
@@
     (pin "8")
     (instances
-      (project "pi_flux_r3_wiring"
+      (project "ktemata_r3_wiring"
         (path "/9545ffa8-4da6-4e23-961a-0f1b69dedae2"
           (reference "J6")
@@
   (label "BATT_4S_N" (at 44.45 226.06 180) (effects (font (size 2 2)) (justify right bottom)))
   (symbol
-    (lib_id "PiFlux:PI5")
+    (lib_id "Ktemata:PI5")
     (at 170.18 55.88 0)
     (unit 1)
@@
     (pin "8")
     (instances
-      (project "pi_flux_r3_wiring"
+      (project "ktemata_r3_wiring"
         (path "/9545ffa8-4da6-4e23-961a-0f1b69dedae2"
           (reference "J7")
@@
   (no_connect (at 165.1 66.04))
   (symbol
-    (lib_id "PiFlux:DISPLAY")
+    (lib_id "Ktemata:DISPLAY")
     (at 170.18 100.33 0)
     (unit 1)
@@
     (pin "2")
     (instances
-      (project "pi_flux_r3_wiring"
+      (project "ktemata_r3_wiring"
         (path "/9545ffa8-4da6-4e23-961a-0f1b69dedae2"
           (reference "J8")
@@
   (label "GND" (at 154.94 102.87 180) (effects (font (size 2 2)) (justify right bottom)))
   (symbol
-    (lib_id "PiFlux:NVME")
+    (lib_id "Ktemata:NVME")
     (at 170.18 125.73 0)
     (unit 1)
@@
     (pin "2")
     (instances
-      (project "pi_flux_r3_wiring"
+      (project "ktemata_r3_wiring"
         (path "/9545ffa8-4da6-4e23-961a-0f1b69dedae2"
           (reference "J9")
@@
   (label "GND" (at 154.94 128.27 180) (effects (font (size 2 2)) (justify right bottom)))
   (symbol
-    (lib_id "PiFlux:KEYBOARD")
+    (lib_id "Ktemata:KEYBOARD")
     (at 170.18 151.13 0)
     (unit 1)
@@
     (pin "2")
     (instances
-      (project "pi_flux_r3_wiring"
+      (project "ktemata_r3_wiring"
         (path "/9545ffa8-4da6-4e23-961a-0f1b69dedae2"
           (reference "J10")
@@
   (label "GND" (at 154.94 153.67 180) (effects (font (size 2 2)) (justify right bottom)))
   (symbol
-    (lib_id "PiFlux:PI_RTC")
+    (lib_id "Ktemata:PI_RTC")
     (at 170.18 176.53 0)
     (unit 1)
@@
     (pin "2")
     (instances
-      (project "pi_flux_r3_wiring"
+      (project "ktemata_r3_wiring"
         (path "/9545ffa8-4da6-4e23-961a-0f1b69dedae2"
           (reference "J11")
@@
   (label "GND" (at 154.94 179.07 180) (effects (font (size 2 2)) (justify right bottom)))
   (symbol
-    (lib_id "PiFlux:FB")
+    (lib_id "Ktemata:FB")
     (at 300.99 55.88 0)
     (unit 1)
@@
     (pin "8")
     (instances
-      (project "pi_flux_r3_wiring"
+      (project "ktemata_r3_wiring"
         (path "/9545ffa8-4da6-4e23-961a-0f1b69dedae2"
           (reference "J12")
@@
   (label "GND" (at 285.75 66.04 180) (effects (font (size 2 2)) (justify right bottom)))
   (symbol
-    (lib_id "PiFlux:OLED")
+    (lib_id "Ktemata:OLED")
     (at 300.99 105.41 0)
     (unit 1)
@@
     (pin "4")
     (instances
-      (project "pi_flux_r3_wiring"
+      (project "ktemata_r3_wiring"
         (path "/9545ffa8-4da6-4e23-961a-0f1b69dedae2"
           (reference "J13")
@@
   (label "I2C_SCL" (at 285.75 110.49 180) (effects (font (size 2 2)) (justify right bottom)))
   (symbol
-    (lib_id "PiFlux:BME")
+    (lib_id "Ktemata:BME")
     (at 300.99 135.89 0)
     (unit 1)
@@
     (pin "4")
     (instances
-      (project "pi_flux_r3_wiring"
+      (project "ktemata_r3_wiring"
         (path "/9545ffa8-4da6-4e23-961a-0f1b69dedae2"
           (reference "J14")
@@
   (label "I2C_SCL" (at 285.75 140.97 180) (effects (font (size 2 2)) (justify right bottom)))
   (symbol
-    (lib_id "PiFlux:DS3231")
+    (lib_id "Ktemata:DS3231")
     (at 300.99 166.37 0)
     (unit 1)
@@
     (pin "4")
     (instances
-      (project "pi_flux_r3_wiring"
+      (project "ktemata_r3_wiring"
         (path "/9545ffa8-4da6-4e23-961a-0f1b69dedae2"
           (reference "J15")
@@
   (label "I2C_SCL" (at 285.75 171.45000000000002 180) (effects (font (size 2 2)) (justify right bottom)))
   (symbol
-    (lib_id "PiFlux:TRACK")
+    (lib_id "Ktemata:TRACK")
     (at 300.99 196.85 0)
     (unit 1)
@@
     (pin "4")
     (instances
-      (project "pi_flux_r3_wiring"
+      (project "ktemata_r3_wiring"
         (path "/9545ffa8-4da6-4e23-961a-0f1b69dedae2"
           (reference "J16")
@@
   (label "I2C_SCL" (at 285.75 201.93 180) (effects (font (size 2 2)) (justify right bottom)))
   (symbol
-    (lib_id "PiFlux:BUTTON")
+    (lib_id "Ktemata:BUTTON")
     (at 300.99 227.33 0)
     (unit 1)
@@
     (pin "2")
     (instances
-      (project "pi_flux_r3_wiring"
+      (project "ktemata_r3_wiring"
         (path "/9545ffa8-4da6-4e23-961a-0f1b69dedae2"
           (reference "J17")
